File: usb_pd_pico_controller/usb_pd_pico_controller.kicad_pcb (KiCad board)
At the start: 2 copper layers, 120 x 100 mm, 64 parts, among them J1 LCSC C145956, J2 LCSC C145956, J3 Conn_01x26_Socket, J4 Conn_01x26_Socket, J5 USB_C_Receptacle_USB2.0_16P, J6 Conn_01x20_Socket, J7 Conn_01x20_Socket, Q1 STL6P3LLH6, SW1 TS5220A, U1 STUSB4531QTR, U2 AP63203WU, U3 AP63203WU, U4 AP63203WU, U5 AP63203WU

Commit message: Consolidated BOM item (100nF)
Signed-off-by: Thomas Flummer <tf@flummer.net>
Parts:
- C4: value 100nF -> 100nF, X5R/X7R, 50V
Changed lines of the file:
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@@
 			)
 		)
-		(property "Value" "100nF"
+		(property "Value" "100nF, X5R/X7R, 50V"
 			(at 0 1.43 0)
 			(layer "F.Fab")
@@
 			)
 		)
-		(attr through_hole)
+		(attr board_only exclude_from_pos_files exclude_from_bom)
 		(duplicate_pad_numbers_are_jumpers no)
 		(fp_poly
